File: TI994A_PSU_Replacement/TI994A_PSU_Replacement.kicad_sch (KiCad schematic)
At the start: 19 parts, among them J1 Power In, J2 Power Out, Q1 SUP53P06-20-E3, SW1 SW_Slide_DPDT, U1 R-78CK5.0-0.5, U2 DFR0831

Commit message: Added BOM
Parts:
- SW1: Manufacturer_Name (none) -> G-Switch Electronic Technology
- U2: Manufacturer_Name (none) -> DFRobot
Changed lines of the file:
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@@
 			)
 		)
-		(property "Datasheet" "~"
+		(property "Datasheet" "https://www.lcsc.com/datasheet/C2848925.pdf"
 			(at 53.34 43.18 0)
 			(effects
@@
 		)
 		(property "Description" "Slide Switch, dual pole double throw"
+			(at 53.34 43.18 0)
+			(effects
+				(font
+					(size 1.27 1.27)
+				)
+				(hide yes)
+			)
+		)
+		(property "Manufacturer_Name" "G-Switch Electronic Technology"
 			(at 53.34 43.18 0)
 			(effects
@@
 			)
 		)
-		(property "Datasheet" ""
+		(property "Datasheet" "https://www.mouser.com/pdfDocs/Product_Overview-DFRobot-DC-DCBuckConverter1.pdf?_gl=1*10lv6ib*_gcl_au*MTIwMTI3ODUxMy4xNzYxNjI0NTM3LjE5MjU4NTE2NTEuMTc2MTk3NTk4Mi4xNzYxOTc1OTgx*_ga*ODY1NjA4MjI5LjE3NjE2MjQ1Mzg.*_ga_15W4STQT4T*czE3NjE5NzU5NzUkbzgkZzEkdDE3NjE5NzYwMDUkajMwJGwwJGgw"
 			(at 152.4 30.48 0)
 			(effects
@@
 			)
 		)
-		(property "Description" "DC-DC Buck Converter"
+		(property "Description" "DC-DC Buck Converter 7-24V to 5V 4A"
 			(at 152.4 30.48 0)
 			(effects
+				(font
+					(size 1.27 1.27)
+				)
+				(hide yes)
+			)
+		)
+		(property "Manufacturer_Name" "DFRobot"
+			(at 152.4 30.48 0)
+			(effects
